Commit message: Functional AMCL

File: my_robot/urdf/my_robot.xacro (robot description, xacro)
@@ -24,5 +24,5 @@
     <inertial>
       <mass value="20.0"/>
-      <origin xyz="0.0 0 0" rpy=" 0 0 0"/>
+      <origin xyz="0.0 0 0.1" rpy=" 0 0 0"/>
       <inertia
           ixx="0.1" ixy="0" ixz="0"

Commit message: fix: robot appearing under map in rviz

File: my_robot/urdf/my_robot.xacro (robot description, xacro)
@@ -16,5 +16,5 @@
   <link name="robot_footprint"></link>
   <joint name="robot_footprint_joint" type="fixed">
-    <origin xyz="0 0 0" rpy="0 0 0" />
+    <origin xyz="0 0 0.1" rpy="0 0 0" />
     <parent link="robot_footprint"/>
     <child link="chassis" />
@@ -24,5 +24,5 @@
     <inertial>
       <mass value="20.0"/>
-      <origin xyz="0.0 0 0.1" rpy=" 0 0 0"/>
+      <origin xyz="0.0 0 0" rpy=" 0 0 0"/>
       <inertia
           ixx="0.1" ixy="0" ixz="0"

Commit message: Added RGB-D camera

File: my_robot/urdf/my_robot.xacro (robot description, xacro)
@@ -159,4 +159,11 @@
     <axis xyz="0 1 0" rpy="0 0 0"/>
   </joint>
+  <joint name="camera_optical_joint" type="fixed">
+    <origin xyz="0 0 0" rpy="-1.5707 0 -1.5707"/>
+    <parent link="camera"/>
+    <child link="camera_link_optical"/>
+  </joint>
+  <link name="camera_link_optical">
+  </link>
   <link name='hokuyo'>
     <inertial>
